Commit message: usd style new asset

File: active_adaptation/assets/unitree_description/urdf/g1/main.urdf (robot description, URDF)
Before this commit: robot g1, 40 links, 39 joints
Links:
- link head_link: geometry visual mesh filename=/home/pjlab/active-adaptation/active_adaptation/assets/unit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
- link left_ankle_pitch_link: geometry visual mesh filename=/home/pjlab/active-adaptation/active_adaptation/assets/unit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
- link left_ankle_roll_link: geometry collision cylinder length=0.05 radius=0.01; collision cylinder length=0.05 radius=0.01
- link left_elbow_link: geometry collision cylinder length=0.13 radius=0.035; visual mesh filename=/home/pjlab/active-adaptation/active_adaptation/assets/unit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
- link left_hip_pitch_link: geometry visual mesh filename=/home/pjlab/active-adaptation/active_adaptation/assets/unit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
- link left_hip_roll_link: geometry collision cylinder length=0.2 radius=0.05; visual mesh filename=/home/pjlab/active-adaptation/active_adaptation/assets/unit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
- link left_hip_yaw_link: geometry visual mesh filename=/home/pjlab/active-adaptation/active_adaptation/assets/unit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
- link left_knee_link: geometry collision cylinder length=0.2 radius=0.05; visual mesh filename=/home/pjlab/active-adaptation/active_adaptation/assets/unit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
- link left_rubber_hand: geometry visual mesh filename=/home/pjlab/active-adaptation/active_adaptation/assets/unit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
- link left_shoulder_pitch_link: geometry visual mesh filename=/home/pjlab/active-adaptation/active_adaptation/assets/unit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
- link left_shoulder_roll_link: geometry visual mesh filename=/home/pjlab/active-adaptation/active_adaptation/assets/unit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
- link left_shoulder_yaw_link: geometry collision cylinder length=0.13 radius=0.035; visual mesh filename=/home/pjlab/active-adaptation/active_adaptation/assets/unit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
- link left_wrist_pitch_link: geometry visual mesh filename=/home/pjlab/active-adaptation/active_adaptation/assets/unit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
- link left_wrist_roll_link: geometry visual mesh filename=/home/pjlab/active-adaptation/active_adaptation/assets/unit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
- link left_wrist_yaw_link: geometry collision cylinder length=0.05 radius=0.05; visual mesh filename=/home/pjlab/active-adaptation/active_adaptation/assets/unit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
- link logo_link: geometry visual mesh filename=/home/pjlab/active-adaptation/active_adaptation/assets/unit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
- link pelvis: geometry collision sphere radius=0.07; visual mesh filename=/home/pjlab/active-adaptation/active_adaptation/assets/unit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
- link pelvis_contour_link: geometry visual mesh filename=/home/pjlab/active-adaptation/active_adaptation/assets/unit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
- link right_ankle_pitch_link: geometry visual mesh filename=/home/pjlab/active-adaptation/active_adaptation/assets/unit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
- link right_ankle_roll_link: geometry collision cylinder length=0.05 radius=0.01; collision cylinder length=0.05 radius=0.01
- link right_elbow_link: geometry collision cylinder length=0.13 radius=0.035; visual mesh filename=/home/pjlab/active-adaptation/active_adaptation/assets/unit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
- link right_hip_pitch_link: geometry visual mesh filename=/home/pjlab/active-adaptation/active_adaptation/assets/unit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
- link right_hip_roll_link: geometry collision cylinder length=0.2 radius=0.05; visual mesh filename=/home/pjlab/active-adaptation/active_adaptation/assets/unit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
- link right_hip_yaw_link: geometry visual mesh filename=/home/pjlab/active-adaptation/active_adaptation/assets/unit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
- link right_knee_link: geometry collision cylinder length=0.2 radius=0.05; visual mesh filename=/home/pjlab/active-adaptation/active_adaptation/assets/unit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
- link right_rubber_hand: geometry visual mesh filename=/home/pjlab/active-adaptation/active_adaptation/assets/unit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
- link right_shoulder_pitch_link: geometry visual mesh filename=/home/pjlab/active-adaptation/active_adaptation/assets/unit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
- link right_shoulder_roll_link: geometry visual mesh filename=/home/pjlab/active-adaptation/active_adaptation/assets/unit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
- link right_shoulder_yaw_link: geometry collision cylinder length=0.13 radius=0.035; visual mesh filename=/home/pjlab/active-adaptation/active_adaptation/assets/unit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
- link right_wrist_pitch_link: geometry visual mesh filename=/home/pjlab/active-adaptation/active_adaptation/assets/unit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
- link right_wrist_roll_link: geometry visual mesh filename=/home/pjlab/active-adaptation/active_adaptation/assets/unit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
- link right_wrist_yaw_link: geometry collision cylinder length=0.05 radius=0.05; visual mesh filename=/home/pjlab/active-adaptation/active_adaptation/assets/unit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
- link torso_link: geometry collision cylinder length=0.01 radius=0.068; collision cylinder length=0.04 radius=0.065
- link waist_roll_link: geometry visual mesh filename=/home/pjlab/active-adaptation/active_adaptation/assets/unit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
- link waist_yaw_link: geometry visual mesh filename=/home/pjlab/active-adaptation/active_adaptation/assets/unit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

Commit message: update w/ new collision

File: active_adaptation/assets/unitree_description/urdf/g1/main.urdf (robot description, URDF)
Before this commit: robot g1, 40 links, 39 joints
Links:
- link left_ankle_roll_link: geometry collision mesh filename=/home/pjlab/active-adaptation/active_adaptation/assets/unit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; visual mesh filename=/home/pjlab/active-adaptation/active_adaptation/assets/unit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
- link left_rubber_hand: geometry collision cylinder length=0.12 radius=0.04; visual mesh filename=/home/pjlab/active-adaptation/active_adaptation/assets/unit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
- link left_wrist_yaw_link: geometry collision cylinder length=0.05 radius=0.035; visual mesh filename=/home/pjlab/active-adaptation/active_adaptation/assets/unit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
- link right_ankle_roll_link: geometry collision mesh filename=/home/pjlab/active-adaptation/active_adaptation/assets/unit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; visual mesh filename=/home/pjlab/active-adaptation/active_adaptation/assets/unit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
- link right_rubber_hand: geometry collision cylinder length=0.12 radius=0.04; visual mesh filename=/home/pjlab/active-adaptation/active_adaptation/assets/unit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
- link right_wrist_yaw_link: geometry collision cylinder length=0.05 radius=0.035; visual mesh filename=/home/pjlab/active-adaptation/active_adaptation/assets/unit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
- link torso_link: geometry collision cylinder length=0.26 radius=0.1; collision sphere length=0.15 radius=0.08

Commit message: mujoco w/ trimesh scan

File: active_adaptation/assets/unitree_description/urdf/g1/main.urdf (robot description, URDF)
Before this commit: robot g1, 40 links, 39 joints
Links:
- link head_link: geometry visual mesh filename=/home/elgce/active-adaptation/active_adaptation/assets/unit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
- link left_ankle_pitch_link: geometry visual mesh filename=/home/elgce/active-adaptation/active_adaptation/assets/unit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
- link left_ankle_roll_link: geometry collision mesh filename=/home/elgce/active-adaptation/active_adaptation/assets/unit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; visual mesh filename=/home/elgce/active-adaptation/active_adaptation/assets/unit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
- link left_elbow_link: geometry collision cylinder length=0.13 radius=0.035; visual mesh filename=/home/elgce/active-adaptation/active_adaptation/assets/unit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
- link left_hip_pitch_link: geometry visual mesh filename=/home/elgce/active-adaptation/active_adaptation/assets/unit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
- link left_hip_roll_link: geometry collision cylinder length=0.2 radius=0.05; visual mesh filename=/home/elgce/active-adaptation/active_adaptation/assets/unit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
- link left_hip_yaw_link: geometry visual mesh filename=/home/elgce/active-adaptation/active_adaptation/assets/unit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
- link left_knee_link: geometry collision cylinder length=0.2 radius=0.05; visual mesh filename=/home/elgce/active-adaptation/active_adaptation/assets/unit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
- link left_rubber_hand: geometry collision cylinder length=0.12 radius=0.04; visual mesh filename=/home/elgce/active-adaptation/active_adaptation/assets/unit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
- link left_shoulder_pitch_link: geometry visual mesh filename=/home/elgce/active-adaptation/active_adaptation/assets/unit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
- link left_shoulder_roll_link: geometry visual mesh filename=/home/elgce/active-adaptation/active_adaptation/assets/unit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
- link left_shoulder_yaw_link: geometry collision cylinder length=0.13 radius=0.035; visual mesh filename=/home/elgce/active-adaptation/active_adaptation/assets/unit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
- link left_wrist_pitch_link: geometry visual mesh filename=/home/elgce/active-adaptation/active_adaptation/assets/unit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
- link left_wrist_roll_link: geometry visual mesh filename=/home/elgce/active-adaptation/active_adaptation/assets/unit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
- link left_wrist_yaw_link: geometry collision cylinder length=0.05 radius=0.035; visual mesh filename=/home/elgce/active-adaptation/active_adaptation/assets/unit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
- link logo_link: geometry visual mesh filename=/home/elgce/active-adaptation/active_adaptation/assets/unit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
- link pelvis: geometry collision sphere radius=0.07; visual mesh filename=/home/elgce/active-adaptation/active_adaptation/assets/unit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
- link pelvis_contour_link: geometry visual mesh filename=/home/elgce/active-adaptation/active_adaptation/assets/unit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
- link right_ankle_pitch_link: geometry visual mesh filename=/home/elgce/active-adaptation/active_adaptation/assets/unit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
- link right_ankle_roll_link: geometry collision mesh filename=/home/elgce/active-adaptation/active_adaptation/assets/unit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; visual mesh filename=/home/elgce/active-adaptation/active_adaptation/assets/unit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
- link right_elbow_link: geometry collision cylinder length=0.13 radius=0.035; visual mesh filename=/home/elgce/active-adaptation/active_adaptation/assets/unit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
- link right_hip_pitch_link: geometry visual mesh filename=/home/elgce/active-adaptation/active_adaptation/assets/unit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
- link right_hip_roll_link: geometry collision cylinder length=0.2 radius=0.05; visual mesh filename=/home/elgce/active-adaptation/active_adaptation/assets/unit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
- link right_hip_yaw_link: geometry visual mesh filename=/home/elgce/active-adaptation/active_adaptation/assets/unit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
- link right_knee_link: geometry collision cylinder length=0.2 radius=0.05; visual mesh filename=/home/elgce/active-adaptation/active_adaptation/assets/unit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
- link right_rubber_hand: geometry collision cylinder length=0.12 radius=0.04; visual mesh filename=/home/elgce/active-adaptation/active_adaptation/assets/unit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
- link right_shoulder_pitch_link: geometry visual mesh filename=/home/elgce/active-adaptation/active_adaptation/assets/unit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
- link right_shoulder_roll_link: geometry visual mesh filename=/home/elgce/active-adaptation/active_adaptation/assets/unit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
- link right_shoulder_yaw_link: geometry collision cylinder length=0.13 radius=0.035; visual mesh filename=/home/elgce/active-adaptation/active_adaptation/assets/unit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
- link right_wrist_pitch_link: geometry visual mesh filename=/home/elgce/active-adaptation/active_adaptation/assets/unit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
- link right_wrist_roll_link: geometry visual mesh filename=/home/elgce/active-adaptation/active_adaptation/assets/unit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
- link right_wrist_yaw_link: geometry collision cylinder length=0.05 radius=0.035; visual mesh filename=/home/elgce/active-adaptation/active_adaptation/assets/unit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
- link torso_link: geometry collision cylinder length=0.26 radius=0.1; collision sphere length=0.15 radius=0.08
- link waist_roll_link: geometry visual mesh filename=/home/elgce/active-adaptation/active_adaptation/assets/unit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
- link waist_yaw_link: geometry visual mesh filename=/home/elgce/active-adaptation/active_adaptation/assets/unit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
